Commit message: correct physics

File: src/yatabot/urdf/yatabot.urdf.xacro (robot description, xacro)
@@ -24,4 +24,10 @@
                 </inertial>
         </xacro:macro>
+        <xacro:macro name="wheel_inertial" params="mass r h">
+                <inertial>
+                        <mass value="${mass}" />
+                        <inertia ixx="${mass*(3*r*r+h*h)/12}" ixy="0.0" ixz="0.0" iyy="${mass*(3*r*r+h*h)/12}" iyz="0.0" izz="${mass*r*r/2}" />
+                </inertial>
+        </xacro:macro>
         <link name="base_link">
                 <visual>
@@ -34,10 +40,10 @@
                 <collision>
                         <geometry>
-				<box size="${width} ${length} ${height}" />
+				<box size="${width-wheelark_depth*2} ${length} ${height}" />
                         </geometry>
                 </collision>
                 <inertial>
-                        <mass value="1.2" />
-                        <origin xyz="0.05 0 0" />
+                        <mass value="1.5" />
+                        <origin xyz="-0.02 0 0" />
                         <inertia ixx="1.0" ixy="0.0" ixz="0.0" iyy="1.0" iyz="0.0" izz="1.0" />
                 </inertial>
@@ -58,5 +64,5 @@
                                 </geometry>
                         </collision>
-                        <xacro:default_inertial mass="0.2" />
+                        <xacro:wheel_inertial mass="0.3" r="${wheeldiam/6}" h="${wheelwidth}" />
                 </link>
                 <joint name="${prefix}_wheel_joint" type="continuous">
@@ -67,8 +73,10 @@
                 </joint>
                 <gazebo reference="${prefix}_wheel">
-                        <mu1 value="200.0" />
-                        <mu2 value="100.0" />
+                        <mu1 value="1.0" />
+                        <mu2 value="1.0" />
                         <kp value="1000000.0" />
                         <kd value="1.0" />
+                        <maxVel>0.0</maxVel>
+                        <minDepth>0.001</minDepth>
                         <material>Gazebo/Grey</material>
                 </gazebo>
@@ -97,10 +105,24 @@
                         </geometry>
                 </collision>
-                <xacro:default_inertial mass="0.05" />
+                <xacro:default_inertial mass="0.08" />
         </link>
         <joint name="caster_joint" type="fixed">
                 <parent link="base_link" />
                 <child link="caster" />
-                <origin xyz="0.06 0 -${height/2+clearance-caster_diam/2}" rpy="0 0 0"/>
+                <origin xyz="-0.06 0 -${height/2+clearance-caster_diam/2}" rpy="0 0 0"/>
         </joint>
+        <gazebo reference="caster">
+                <mu1 value="0.01" />
+                <mu2 value="0.01" />
+                <kp value="1000000.0" />
+                <kd value="1.0" />
+                <maxVel>0.0</maxVel>
+                <minDepth>0.001</minDepth>
+                <material>Gazebo/Grey</material>
+        </gazebo>
+        <gazebo>
+                <plugin name="gazebo_ros_control" filename="libgazebo_ros_control.so">
+                        <robotNamespace>/</robotNamespace>
+                </plugin>
+        </gazebo>
 </robot>

Commit message: wheel model

File: src/yatabot/urdf/yatabot.urdf.xacro (robot description, xacro)
@@ -52,9 +52,8 @@
                 <link name="${prefix}_wheel">
                         <visual>
-                                <origin xyz="0 0 0" rpy="${pi/2} 0 0 " />
+                                <origin xyz="0 0 0" rpy="0 0 ${pi/2} " />
                                 <geometry>
-                                        <cylinder radius="${wheeldiam/2}" length="${wheelwidth}" />
+                                        <mesh filename="package://yatabot/meshes/wheel.dae" />
                                 </geometry>
-                                <material name="black" />
                         </visual>
                         <collision>

Commit message: cam_tracker

File: src/yatabot/urdf/yatabot.urdf.xacro (robot description, xacro)
@@ -12,4 +12,5 @@
         <xacro:property name="wheelwidth" value="0.015" />
         <xacro:property name="pi" value="3.141592" />
+        <xacro:property name="camera_link" value="0.02" />
         <material name="white">
                 <color rgba="1 1 1 1" />
@@ -40,5 +41,5 @@
                 <collision>
                         <geometry>
-				<box size="${width-wheelark_depth*2} ${length} ${height}" />
+        <box size="${width-wheelark_depth*2} ${length} ${height}" />
                         </geometry>
                 </collision>
@@ -90,6 +91,6 @@
                 </transmission>
         </xacro:macro>
-	<xacro:wheel prefix="left" base="base_link" reflect="1" />
-        <xacro:wheel prefix="right" base="base_link" reflect="-1" />
+  <xacro:wheel prefix="left" base="base_link" reflect="1" />
+  <xacro:wheel prefix="right" base="base_link" reflect="-1" />
         <link name="caster">
                 <visual>
@@ -124,4 +125,70 @@
                         <robotNamespace>/</robotNamespace>
                 </plugin>
-        </gazebo>
+              </gazebo>
+  <joint name="camera_joint" type="fixed">
+    <axis xyz="0 1 0" />
+    <origin xyz="${length/2 - camera_link/2} 0 ${height/2 + camera_link/2}" rpy="0 0 0"/>
+    <parent link="base_link"/>
+    <child link="camera_link"/>
+  </joint>
+  <!-- Camera -->
+  <link name="camera_link">
+    <collision>
+      <origin xyz="0 0 0" rpy="0 0 0"/>
+      <geometry>
+    <box size="${camera_link} ${camera_link} ${camera_link}"/>
+      </geometry>
+    </collision>
+    <visual>
+      <origin xyz="0 0 0" rpy="0 0 0"/>
+      <geometry>
+    <box size="${camera_link} ${camera_link} ${camera_link}"/>
+      </geometry>
+      <material name="red"/>
+    </visual>
+    <inertial>
+      <mass value="1e-5" />
+      <origin xyz="0 0 0" rpy="0 0 0"/>
+      <inertia ixx="1e-6" ixy="0" ixz="0" iyy="1e-6" iyz="0" izz="1e-6" />
+    </inertial>
+  </link>
+   <gazebo reference="camera_link">
+    <sensor type="camera" name="camera1">
+      <update_rate>30.0</update_rate>
+      <camera name="head">
+        <horizontal_fov>1.3962634</horizontal_fov>
+        <image>
+          <width>800</width>
+          <height>800</height>
+          <format>R8G8B8</format>
+        </image>
+        <clip>
+          <near>0.02</near>
+          <far>300</far>
+        </clip>
+        <noise>
+          <type>gaussian</type>
+          <!-- Noise is sampled independently per pixel on each frame.
+               That pixel's noise value is added to each of its color
+               channels, which at that point lie in the range [0,1]. -->
+          <mean>0.0</mean>
+          <stddev>0.007</stddev>
+        </noise>
+      </camera>
+      <plugin name="camera_controller" filename="libgazebo_ros_camera.so">
+        <alwaysOn>true</alwaysOn>
+        <updateRate>0.0</updateRate>
+        <cameraName>yatabot/camera1</cameraName>
+        <imageTopicName>image_raw</imageTopicName>
+        <cameraInfoTopicName>camera_info</cameraInfoTopicName>
+        <frameName>camera_link</frameName>
+        <hackBaseline>0.07</hackBaseline>
+        <distortionK1>0.0</distortionK1>
+        <distortionK2>0.0</distortionK2>
+        <distortionK3>0.0</distortionK3>
+        <distortionT1>0.0</distortionT1>
+        <distortionT2>0.0</distortionT2>
+      </plugin>
+    </sensor>
+  </gazebo>
 </robot>
